Commit message: Moved "pose publishing" in its own function  * vaious tests to solve TF propagation latency

File: zed_wrapper/urdf/zedm.urdf (robot description, URDF)
Before this commit: robot zedm_camera, 6 links, 5 joints
Links:
- link zed_camera_center: geometry visual box size=0.015 0.125 0.025
- link zed_left_camera_frame: geometry visual cylinder length=0.030 radius=0.01
- link zed_right_camera_frame: geometry visual cylinder length=0.030 radius=0.01
