Commit message: Managed lifecycle launch file working Fixed path in urdf model to load mesh

File: zed_wrapper/urdf/zed.urdf (robot description, URDF)
Before this commit: robot zed_camera, 6 links, 5 joints
Links:
- link zed_camera_center: geometry visual mesh filename=package://stereolabs_zed/urdf/models/ZED.stl

File: zed_wrapper/urdf/zedm.urdf (robot description, URDF)
Before this commit: robot zedm_camera, 6 links, 5 joints
Links:
- link zed_camera_center: geometry visual mesh filename=package://stereolabs_zed/urdf/models/ZEDM.stl
- link zed_left_camera_frame: geometry 
- link zed_right_camera_frame: geometry 
